Commit message: updates

File: assets/kuka_iiwa.urdf (robot description, URDF)
Before this commit: robot lbr_iiwa, 8 links, 7 joints
Links:
- link lbr_iiwa_link_7: geometry collision mesh filename=meshes/link_7m.stl; visual mesh filename=meshes/link_7m.obj
Joints:
- joint lbr_iiwa_joint_7: origin xyz=0 0.081 0 rpy=-1.57079632679 3.14159265359 0 -> xyz=0 0 0 rpy=-1.57079632679 3.14159265359 0
